File: template-project.kicad_pcb (KiCad board)
At the start: 2 copper layers, 0 parts

Commit message: Added medium and small chof logo
Parts:
- added G***: LOGO, LOGO, B.Cu at (30.5, 184.9)
- added G***: LOGO, LOGO, B.Cu at (22.4, 182.3)

Commit message: Updated template for KiCAD 7
Parts:
- G***: footprint LOGO -> Chof747 Logos:LOGO small
